Commit message: feat(dual_arm_base_description): update robot description and controllers
- Added dual_arm_base_description to settings.json for visualization.
- Simplified controller.launch by removing unused position controllers.
- Cleaned up controller.yaml by removing unnecessary position controllers.
- Updated dual_arm_base.xacro to define joints as fixed instead of revolute.
- Introduced dual_arm_combined.xacro for combined robot description.

File: assets/dual_arm_base_description/urdf/dual_arm_base.xacro (robot description, xacro)
@@ -1,4 +1,5 @@
 <?xml version="1.0" ?>
 <robot name="dual_arm_base" xmlns:xacro="http://www.ros.org/wiki/xacro">
+<xacro:macro name="dual_arm_base" params="">
 <xacro:include filename="$(find dual_arm_base_description)/urdf/materials.xacro" />
 <xacro:include filename="$(find dual_arm_base_description)/urdf/dual_arm_base.trans" />
@@ -74,10 +75,8 @@
   </actuator>
 </transmission>
-<joint name="joint_l_0" type="revolute">
+<joint name="joint_l_0" type="fixed">
   <origin xyz="0.223407 -0.055779 0.945428" rpy="0.030792 -1.221558 2.585226"/>
   <parent link="base_link"/>
   <child link="L_1"/>
-  <axis xyz="0 0 1"/>
-  <limit upper="3.141593" lower="-3.141593" effort="100" velocity="100"/>
 </joint>
 <transmission name="joint_r_0_tran">
@@ -91,10 +90,9 @@
   </actuator>
 </transmission>
-<joint name="joint_r_0" type="revolute">
+<joint name="joint_r_0" type="fixed">
   <origin xyz="-0.223407 -0.055779 0.945428" rpy="-0.030792 -1.221558 0.556367"/>
   <parent link="base_link"/>
   <child link="R_1"/>
-  <axis xyz="0 0 1"/>
-  <limit upper="3.141593" lower="-3.141593" effort="100" velocity="100"/>
 </joint>
+</xacro:macro>
 </robot>
