Commit message: Remove obsolete files and add new URDF/XACRO for dual arm base description
- Deleted the old base_link.STL mesh file.
- Removed the outdated dual_arm_base.trans transmission file.
- Introduced a new dual_arm_base.urdf.xacro file containing the complete robot description, including links, joints, and visual/collision geometries.

File: assets/dual_arm_base_description/urdf/materials.xacro (robot description, xacro)
@@ -1,6 +1,6 @@
 <?xml version="1.0" ?>
-<robot name="dual_arm_base" xmlns:xacro="http://www.ros.org/wiki/xacro" >
-<material name="silver">
-  <color rgba="0.700 0.700 0.700 1.000"/>
-</material>
+<robot xmlns:xacro="http://www.ros.org/wiki/xacro" name="dual_arm_base">
+  <material name="silver">
+    <color rgba="0.700 0.700 0.700 1.000"/>
+  </material>
 </robot>

File: assets/dual_arm_description/urdf/dual_arm_combined.xacro (robot description, xacro)
@@ -1,13 +1,3 @@
 <?xml version="1.0" ?>
-<!--
-  Dual Arm Combined Robot Description (XACRO)
-  This file defines a dual-arm robotic system combining:
-  - A central base platform (dual_arm base)
-  - Two Nova2 robotic arms (left and right)
-  The system is designed for dual-arm manipulation tasks with synchronized
-  or independent control of both manipulators.
-  Author: Generated for dual-teleop-viz project
-  Date: September 2025
--->
 <robot name="dual_arm_combined" xmlns:xacro="http://www.ros.org/wiki/xacro">
   <!-- ========================================================================= -->
@@ -20,9 +10,8 @@
   <!-- ========================================================================= -->
   <!-- Include base platform description -->
-  <xacro:include filename="$(find dual_arm_description)/urdf/dual_arm_base.xacro" />
+  <xacro:include filename="$(find dual_arm_base_description)/urdf/dual_arm_base.urdf.xacro" />
   <!-- Include Nova2 robot arm description -->
-  <xacro:include filename="$(find dual_arm_description)/urdf/nova2_robot.xacro" />
+  <xacro:include filename="$(find dobot_rviz)/urdf/nova2_robot.xacro" />
   <!-- Include materials definitions -->
-  <xacro:include filename="$(find dual_arm_description)/urdf/materials.xacro" />
   <!-- ========================================================================= -->
   <!-- MAIN ROBOT MACRO DEFINITION -->
@@ -35,11 +24,9 @@
     <!-- Nova2 robotic arm mounted on the left side of the base platform -->
     <xacro:nova2_robot
-      prefix="left_"
-      base_link_name="left_base"/>
+      prefix="left_" />
     <!-- Right arm instantiation -->
     <!-- Nova2 robotic arm mounted on the right side of the base platform -->
     <xacro:nova2_robot
-      prefix="right_"
-      base_link_name="right_base"/>
+      prefix="right_" />
     <!-- Joint connecting left arm to base platform -->
     <joint name="left_arm_base_joint" type="fixed">
