Commit message: feat(nova2_robot): enhance robot description with detailed properties
- Added inertial, visual, and collision elements for each link in the nova2_robot.
- Updated the joint definitions to improve the robot's structure.
- Preserved the original link structure while copying child elements in the converter.

File: assets/dobot_rviz/urdf/nova2_robot.xacro (robot description, xacro)
@@ -209,4 +209,4 @@
     </joint>
   </xacro:macro>
-  <!-- <xacro:nova2_robot prefix="${prefix}" base_link_name="${base_link_name}"/> -->
+  <xacro:nova2_robot prefix="${prefix}" base_link_name="${base_link_name}"/>
 </robot>

File: assets/dual_arm_description/urdf/dual_arm_combined.xacro (robot description, xacro)
@@ -46,5 +46,5 @@
       <parent link="L_1"/>
       <child link="left_dummy_link"/>
-      <origin xyz="0 0 0" rpy="0 0 0"/>
+      <origin xyz="0 0 0" rpy="0 0 ${PI}"/>
     </joint>
     <!-- Joint connecting right arm to base platform -->

Commit message: refactor(dual_arm_base_description): update launch files and robot description
- Removed legacy display.launch file to streamline the codebase.
- Added new display.launch.xml file with updated arguments and nodes.
- Updated dual_arm_combined.xacro to include nova2_robot.xacro from the correct path.
- Simplified nova2_robot macro parameters by removing base_link_name.

File: assets/dobot_rviz/urdf/nova2_robot.xacro (robot description, xacro)
@@ -5,8 +5,7 @@
   <xacro:property name="package_name" value="robot_description"/>
   <xacro:property name="prefix" value=""/>
-  <xacro:property name="base_link_name" value="base_link"/>
-  <xacro:macro name="nova2_robot" params="prefix base_link_name">
+  <xacro:macro name="nova2_robot" params="prefix">
     <link name="${prefix}dummy_link"/>
-    <link name="${prefix}${base_link_name}">
+    <link name="${prefix}base_link">
       <inertial>
         <origin xyz="1.31739324853774E-05 -7.84959718585273E-06 0.0647773077977383" rpy="0 0 0"/>
@@ -164,9 +163,9 @@
     <joint name="${prefix}dummy_joint" type="fixed">
       <parent link="${prefix}dummy_link"/>
-      <child link="${prefix}${base_link_name}"/>
+      <child link="${prefix}base_link"/>
     </joint>
     <joint name="${prefix}joint1" type="revolute">
       <origin xyz="0 0 0.2234" rpy="0 0 0"/>
-      <parent link="${prefix}${base_link_name}"/>
+      <parent link="${prefix}base_link"/>
       <child link="${prefix}Link1"/>
       <axis xyz="0 0 1"/>
@@ -209,4 +208,4 @@
     </joint>
   </xacro:macro>
-  <xacro:nova2_robot prefix="${prefix}" base_link_name="${base_link_name}"/>
+  <!-- <xacro:nova2_robot prefix="${prefix}" /> -->
 </robot>

File: assets/dual_arm_base_description/urdf/dual_arm_combined.xacro (robot description, xacro)
@@ -1,13 +1,3 @@
 <?xml version="1.0" ?>
-<!--
-  Dual Arm Combined Robot Description (XACRO)
-  This file defines a dual-arm robotic system combining:
-  - A central base platform (dual_arm base)
-  - Two Nova2 robotic arms (left and right)
-  The system is designed for dual-arm manipulation tasks with synchronized
-  or independent control of both manipulators.
-  Author: Generated for dual-teleop-viz project
-  Date: September 2025
--->
 <robot name="dual_arm_combined" xmlns:xacro="http://www.ros.org/wiki/xacro">
   <!-- ========================================================================= -->
@@ -22,7 +12,6 @@
   <xacro:include filename="$(find dual_arm_base_description)/urdf/dual_arm_base.xacro" />
   <!-- Include Nova2 robot arm description -->
-  <xacro:include filename="$(find dual_arm_description)/urdf/nova2_robot.xacro" />
+  <xacro:include filename="$(find dobot_rviz)/urdf/nova2_robot.xacro" />
   <!-- Include materials definitions -->
-  <xacro:include filename="$(find dual_arm_description)/urdf/materials.xacro" />
   <!-- ========================================================================= -->
   <!-- MAIN ROBOT MACRO DEFINITION -->
@@ -35,11 +24,9 @@
     <!-- Nova2 robotic arm mounted on the left side of the base platform -->
     <xacro:nova2_robot
-      prefix="left_"
-      base_link_name="left_base"/>
+      prefix="left_" />
     <!-- Right arm instantiation -->
     <!-- Nova2 robotic arm mounted on the right side of the base platform -->
     <xacro:nova2_robot
-      prefix="right_"
-      base_link_name="right_base"/>
+      prefix="right_" />
     <!-- Joint connecting left arm to base platform -->
     <joint name="left_arm_base_joint" type="fixed">
